Commit message: Fixed objects and new labelling scripts

File: kitchen_data_player/urdfs/ias_kitchen.urdf (robot description, URDF)
Before this commit: robot myfirst, 5 links, 4 joints
Links:
- added link countertop_kitchenette; visual box size=2.05 0.575 0.01
- link drawer55: geometry visual box size=0.58 0.78 0.01
Joints:
- added joint countertop_kitchenette_countertop_middle: type fixed, parent countertop_middle, child countertop_kitchenette
